Commit message: pipette visual link

File: config/gazebo_fr3.urdf (robot description, URDF)
Before this commit: robot fr3, 18 links, 17 joints
Links:
- removed link fr3_link8
- added link fr3_link_pip, mass 0.3; visual mesh filename=package://fr3_moveit_config/meshes/visual/link_pip.dae scale=0.001 0.001 0.001
Joints:
- joint fr3_joint8: child fr3_link8 -> fr3_link_pip; origin xyz=0 0 0.107 rpy=0 0 0 -> xyz=0 0 0.107 rpy=0 0 0.785

Commit message: pipette collision

File: config/gazebo_fr3.urdf (robot description, URDF)
Before this commit: robot fr3, 18 links, 17 joints
Links:
- link fr3_link_pip: geometry collision mesh filename=package://fr3_moveit_config/meshes/collision/link_pip.stl scale=0.001 0.001 0.001; visual mesh filename=package://fr3_moveit_config/meshes/visual/link_pip.dae scale=0.001 0.001 0.001
Joints:
- joint fr3_joint8: origin xyz=0 0 0.107 rpy=0 0 0.785 -> xyz=0 0 0.107 rpy=0 0 0.7853981633974483

Commit message: pipette tip link

File: config/gazebo_fr3.urdf (robot description, URDF)
Before this commit: robot fr3, 18 links, 17 joints
Links:
- added link fr3_link_pip_tip
Joints:
- added joint fr3_joint9: type fixed, parent fr3_link_pip, child fr3_link_pip_tip, origin xyz=0 -0.083 0.147997 rpy=0 0 0

Commit message: pip_tip_link reference frame corection

File: config/gazebo_fr3.urdf (robot description, URDF)
Before this commit: robot fr3, 19 links, 18 joints
Joints:
- joint fr3_joint9: origin xyz=0 -0.083 0.147997 rpy=0 0 0 -> xyz=0 -0.083 0.147997 rpy=3.14 0 0
